File: PLC4Uni FelipeLG/OUT-RELAY-2.kicad_sch (KiCad schematic)
At the start: 7 parts, among them K2 Fujitsu_FTR-LYAA005x, Q11 BFN26

Commit message: Add files via upload
Updated Circuitos corregidos y pistas agregadas
Parts:
- removed K2: Fujitsu_FTR-LYAA005x, Relay_THT:Relay_SPST-NO_Fujitsu_FTR-LYAA005x_FormA_Vertical, symbol Relay:Fujitsu_FTR-LYAA005x
- removed OC8: FOD817S, Package_DIP_AKL:SMDIP-4_W9.53mm, symbol Optocoupler_AKL:FOD817S
- removed Q11: BFN26, Package_TO_SOT_SMD_AKL:SOT-23, symbol Transistor_BJT_AKL:BFN26
- removed R36: 2K, Resistor_SMD_AKL:R_0603_1608Metric, symbol Resistor_AKL:R_0603
- removed R37: 10K, Resistor_SMD_AKL:R_0603_1608Metric, symbol Resistor_AKL:R_0603
- removed R38: 510, Resistor_SMD_AKL:R_0603_1608Metric, symbol Resistor_AKL:R_0603
- added K2: G5V-1, Relay_THT:Relay_SPDT_Omron_G5V-1, symbol Relay:G5V-1
- added Q11: DTC123E, Package_TO_SOT_SMD:SOT-23, symbol Transistor_BJT:DTC123E
Connections:
- net GND: now also Q11.2 (E)
- net IN: now also Q11.1 (B)
- net VCC: now also K2.2
- net out-common-2: now also K2.5, K2.6
- net out-no-2: now also K2.10
- net at D3.2 (A): now also K2.9, Q11.3 (C)
- no-connect marks 0 -> 1
