File: PLC4Uni FelipeLG/_autosave-PLC4Uni FelipeLG.kicad_pcb (KiCad board)
At the start: 4 copper layers, 72 parts, among them J1 Power, J2 InPut, J3 OUTNPN, J4 OutNPNOcto, J5 Out-PNP_0-10v, J6 OutPNP, J7 Relay2, J8 RS485, K1 G5V-1, K2 G5V-1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

Commit message: Add files via upload
Updated Circuitos corregidos y pistas agregadas
Routing:
- net /board-plc4uni/input-pnp-1/OUT: track 90.0 -> 0.00 mm, vias 2 -> 0
- net /board-plc4uni/input-npn-1/OUT: track 87.0 -> 0.00 mm, vias 2 -> 0
- net /board-plc4uni/input-npn-opto-2/OUT: track 74.4 -> 0.00 mm, vias 2 -> 0
- net /board-plc4uni/INPUT-0-10V/ADC_IN_3V3: track 63.7 -> 3.19 mm, vias 2 -> 0
- net /board-plc4uni/RS485/UART_RX: track 35.4 -> 0.00 mm, vias 2 -> 0
- net +3.3V: track 143.0 -> 126.8 mm, vias 2 -> 0
- net GND: track 147.1 -> 133.1 mm
- net /board-plc4uni/input-pnp-opto-1/OUT: track 10.1 -> 0.00 mm, vias 1 -> 0
- net /board-plc4uni/input-pnp-2/OUT: track 7.93 -> 0.00 mm, vias 1 -> 0
- net /board-plc4uni/OUTPUT-0-10V/SDA: track 5.09 -> 0.00 mm, vias 1 -> 0
- net /board-plc4uni/input-npn-2/OUT: track 4.89 -> 0.00 mm, vias 1 -> 0
- net /board-plc4uni/input-pnp-opto-2/OUT: track 4.60 -> 0.00 mm, vias 1 -> 0
- net /board-plc4uni/RS485/UART_TX: track 2.13 -> 0.00 mm, vias 1 -> 0
- net /board-plc4uni/OUT-NPN-1/IN: track 2.05 -> 0.00 mm, vias 1 -> 0
- net /board-plc4uni/OUT-RELAY-1/IN: track 2.03 -> 0.00 mm, vias 1 -> 0
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